File: CableHanger.kicad_pcb (KiCad board)
At the start: 2 copper layers, 303 x 303 mm, 0 parts

Commit message: PoC completed
Other:
- board size 303 x 303 mm -> 292 x 292 mm

Commit message: Logo and tool holes added
Parts:
- added Ref**: Val**, SloBloFP:SloBloLogo_123x150, F.Cu at (285.0, 200.0)
Other:
- board size 292 x 292 mm -> 295 x 295 mm
