File: CableHolder.kicad_pcb (KiCad board)
At the start: 2 copper layers, 295 x 295 mm, 9 parts

Commit message: Rename to CableHolder
Other:
- board text added: "SloBlo Labs - Cable Holder ${VERSION}"
- board text removed: "SloBlo Labs - Cable Hanger ${VERSION}"
Changed lines of the file:
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@@
   (paper "A2")
   (title_block
-    (title " Cable Hanger")
+    (title " Cable Holder")
     (date "2023-10-11")
     (rev "${VERSION}")
@@
     (effects (font (size 1 1) (thickness 0.15)) (justify left bottom mirror))
   )
-  (gr_text "SloBlo Labs - Cable Hanger ${VERSION}" (at 430.75 59 90) (layer "B.SilkS")
+  (gr_text "SloBlo Labs - Cable Holder ${VERSION}" (at 430.75 59 90) (layer "B.SilkS")
     (effects (font (size 2 2) (thickness 0.15)) (justify left bottom mirror))
   )
